File: Schematic_PCB/Music_Visualizer/Music_Visualizer.kicad_pcb (KiCad board)
At the start: 2 copper layers, 320 x 175.1 mm, 237 parts, among them J1 AudioJack2_Ground, J2 PJ-079BH, SW1 SW_SPDT, SW2 SW_SPST, U1 LM324, U10 LM3915N-1, U11 LM3915N-1, U12 LM3915N-1, U13 LM3915N-1, U14 LM3915N-1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

Commit message: Added 10 uF polarized smoothing capacitors to LED driver ciruit
Parts:
- removed the C57 at (349.5, 148.0)
- added C59: 10u, Capacitor_THT:CP_Radial_D5.0mm_P2.00mm, F.Cu at (95.0, 108.0)
- added C60: 10u, Capacitor_THT:CP_Radial_D5.0mm_P2.00mm, F.Cu at (135.0, 108.0)
- added C61: 10u, Capacitor_THT:CP_Radial_D5.0mm_P2.00mm, F.Cu at (175.0, 108.0)
- added C62: 10u, Capacitor_THT:CP_Radial_D5.0mm_P2.00mm, F.Cu at (215.0, 108.0)
- added C63: 10u, Capacitor_THT:CP_Radial_D5.0mm_P2.00mm, F.Cu at (255.0, 108.0)
- added C64: 10u, Capacitor_THT:CP_Radial_D5.0mm_P2.00mm, F.Cu at (295.0, 108.0)
- added C65: 10u, Capacitor_THT:CP_Radial_D5.0mm_P2.00mm, F.Cu at (335.0, 108.0)
- renumbered C58 to C57, C59 to C58

Commit message: Changed Grid 1 & 2 to 50 mils and 10 mils respectively, and deleted all traces
Routing:
- net +9V: track 1014.8 -> 0.28 mm
- net Mode: track 264.2 -> 0.00 mm
- net LED_Brightness_Control: track 243.0 -> 1.96 mm, vias 12 -> 0
- net GND: track 97.8 -> 0.57 mm
- net Net-(D61-Pad1): track 46.2 -> 0.00 mm
- net Net-(D51-Pad1): track 46.2 -> 0.00 mm
- net Net-(D41-Pad1): track 46.2 -> 0.00 mm
- net Net-(D31-Pad1): track 46.2 -> 0.00 mm
- net Net-(D21-Pad1): track 46.2 -> 0.00 mm
- net Net-(D11-Pad1): track 46.2 -> 0.00 mm
- net Net-(D1-Pad1): track 46.2 -> 0.00 mm
- net Net-(D30-Pad1): track 35.7 -> 0.00 mm
- net Net-(D40-Pad1): track 35.1 -> 0.00 mm
- net Net-(D70-Pad1): track 33.9 -> 0.00 mm
- net Net-(D60-Pad1): track 33.9 -> 0.00 mm
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- removed copper zone on B.Cu, net GND
Other:
- board text removed: "Brilliance [6kHz:20kHz]"
- board text removed: "Lower-Midrange [250Hz:500Hz]"
- board text removed: "Upper-Midrange [2kHz:4kHz]"

Commit message: Aligned all subcircuits, routed 9V and power, started routing LEDS
Parts:
- moved JP2 98.6 mm to (342.9, 49.5)
- moved SW2 62.0 mm to (299.7, 163.8)
- moved U7 25.5 mm to (321.6, 151.0)
- moved C52 25.1 mm to (332.7, 148.6)
- moved C53 25.0 mm to (328.9, 148.6)
- moved R73 23.7 mm to (321.6, 166.2)
- moved C54 23.5 mm to (308.9, 152.3)
- moved D71 23.5 mm to (331.5, 156.2)
- moved C56 23.1 mm to (328.9, 165.9)
- moved R74 20.8 mm to (335.3, 165.9)
- moved J2 19.3 mm to (352.9, 158.7)
- moved R82 19.0 mm to (337.8, 148.4), turned to 90 degrees
- moved RV1 18.5 mm to (168.9, 176.3)
- moved U17 16.8 mm to (266.7, 171.4)
- moved RV2 15.7 mm to (252.7, 176.3)
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Routing:
- net +9V: track 0.28 -> 843.2 mm
- net /Power/Power: track 0.00 -> 64.3 mm
- net Net-(D70-Pad1): track 0.00 -> 35.9 mm
- net Net-(D60-Pad1): track 0.00 -> 35.9 mm
- net Net-(D40-Pad1): track 0.00 -> 35.9 mm
- net Net-(D30-Pad1): track 0.00 -> 35.9 mm
- net Net-(D20-Pad1): track 0.00 -> 35.9 mm
- net Net-(D50-Pad1): track 0.00 -> 35.9 mm
- net Net-(D10-Pad1): track 1.00 -> 35.9 mm
- net Net-(D9-Pad1): track 0.00 -> 27.5 mm
- net Net-(D19-Pad1): track 0.00 -> 27.5 mm
- net Net-(D29-Pad1): track 0.00 -> 27.5 mm
- net Net-(D69-Pad1): track 0.00 -> 27.5 mm
- net Net-(D59-Pad1): track 0.00 -> 27.5 mm
- net Net-(D39-Pad1): track 0.16 -> 27.5 mm
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Other:
- board size 320 x 175.1 mm -> 295.6 x 157.9 mm
- board text added: "Brilliance [6kHz:20kHz]"
- board text added: "Low-Midrange [250Hz:500Hz]"
- board text added: "Upper-Midrange [2kHz:4kHz]"

Commit message: Finished Routing LEDs
Routing:
- net Net-(D51-Pad1): track 0.00 -> 52.5 mm
- net Net-(D21-Pad1): track 0.00 -> 52.5 mm
- net Net-(D11-Pad1): track 0.00 -> 52.5 mm
- net Net-(D41-Pad1): track 0.00 -> 52.5 mm
- net Net-(D31-Pad1): track 0.00 -> 52.5 mm
- net Net-(D1-Pad1): track 0.00 -> 52.2 mm
- net Net-(D61-Pad1): track 0.00 -> 52.2 mm
- net Net-(D22-Pad1): track 0.00 -> 34.4 mm
- net Net-(D2-Pad1): track 0.00 -> 34.4 mm
- net Net-(D12-Pad1): track 0.00 -> 34.4 mm
- net Net-(D62-Pad1): track 0.00 -> 34.4 mm
- net Net-(D52-Pad1): track 0.00 -> 34.4 mm
- net Net-(D32-Pad1): track 0.00 -> 34.4 mm
- net Net-(D42-Pad1): track 0.00 -> 34.4 mm
- net Net-(D23-Pad1): track 0.00 -> 28.2 mm
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
Commit message: Finieshed Routing Brightness control, FilterOut and RHigh
Routing:
- net LED_Brightness_Control: track 0.00 -> 501.2 mm
- net Rhi_Value: track 0.00 -> 343.2 mm
- net Net-(R80-Pad1): track 0.00 -> 16.5 mm
- net Net-(R79-Pad1): track 0.00 -> 16.5 mm
- net Net-(R77-Pad1): track 0.00 -> 16.5 mm
- net Net-(R76-Pad1): track 0.00 -> 16.5 mm
- net Net-(R75-Pad1): track 0.00 -> 16.5 mm
- net Net-(R78-Pad1): track 0.00 -> 16.5 mm
- net Net-(R81-Pad1): track 0.00 -> 16.5 mm
- net VBrilliance: track 0.00 -> 11.6 mm
- net VUpperMidrange: track 0.00 -> 11.6 mm
- net VPresence: track 0.00 -> 11.6 mm
- net VBass: track 0.00 -> 11.6 mm
- net VSubBass: track 0.00 -> 11.6 mm
- net VMidrange: track 0.00 -> 11.6 mm
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