File: Schematic_PCB/Music_Visualizer/Power.kicad_sch (KiCad schematic)
At the start: 12 parts

Commit message: Completed and annotated Spectrum filters and power circuitry, and updated BOM
Parts:
- gave numbers to parts that had none: 11
Changed lines of the file:
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@@
   (symbol (lib_id "power:+9V") (at 90.17 125.73 0) (unit 1)
     (in_bom yes) (on_board yes) (fields_autoplaced)
-    (property "Reference" "#PWR?" (id 0) (at 90.17 129.54 0)
+    (property "Reference" "#PWR054" (id 0) (at 90.17 129.54 0)
       (effects (font (size 1.27 1.27)) hide)
     )
@@
   (symbol (lib_id "Device:C") (at 60.96 132.08 0) (unit 1)
     (in_bom yes) (on_board yes) (fields_autoplaced)
-    (property "Reference" "C?" (id 0) (at 64.77 130.8099 0)
+    (property "Reference" "C52" (id 0) (at 64.77 130.8099 0)
       (effects (font (size 1.27 1.27)) (justify left))
     )
@@
   (symbol (lib_id "power:GND") (at 67.31 138.43 0) (unit 1)
     (in_bom yes) (on_board yes) (fields_autoplaced)
-    (property "Reference" "#PWR?" (id 0) (at 67.31 144.78 0)
+    (property "Reference" "#PWR053" (id 0) (at 67.31 144.78 0)
       (effects (font (size 1.27 1.27)) hide)
     )
@@
   (symbol (lib_id "Device:C") (at 121.92 134.62 0) (unit 1)
     (in_bom yes) (on_board yes) (fields_autoplaced)
-    (property "Reference" "C?" (id 0) (at 125.73 133.3499 0)
+    (property "Reference" "C54" (id 0) (at 125.73 133.3499 0)
       (effects (font (size 1.27 1.27)) (justify left))
     )
@@
   (symbol (lib_id "Device:C") (at 162.56 54.61 0) (unit 1)
     (in_bom yes) (on_board yes) (fields_autoplaced)
-    (property "Reference" "C?" (id 0) (at 166.37 53.3399 0)
+    (property "Reference" "C50" (id 0) (at 166.37 53.3399 0)
       (effects (font (size 1.27 1.27)) (justify left))
     )
@@
   (symbol (lib_id "Device:C") (at 146.05 138.43 90) (unit 1)
     (in_bom yes) (on_board yes) (fields_autoplaced)
-    (property "Reference" "C?" (id 0) (at 146.05 130.81 90))
+    (property "Reference" "C56" (id 0) (at 146.05 130.81 90))
     (property "Value" "" (id 1) (at 146.05 133.35 90))
     (property "Footprint" "" (id 2) (at 149.86 137.4648 0)
@@
   (symbol (lib_id "Regulator_SwitchedCapacitor:LT1054") (at 109.22 133.35 0) (unit 1)
     (in_bom yes) (on_board yes) (fields_autoplaced)
-    (property "Reference" "U?" (id 0) (at 109.22 118.11 0))
+    (property "Reference" "U7" (id 0) (at 109.22 118.11 0))
     (property "Value" "" (id 1) (at 109.22 120.65 0))
     (property "Footprint" "" (id 2) (at 111.76 135.89 0)
@@
   (symbol (lib_id "Device:C") (at 196.85 54.61 0) (unit 1)
     (in_bom yes) (on_board yes) (fields_autoplaced)
-    (property "Reference" "C?" (id 0) (at 200.66 53.3399 0)
+    (property "Reference" "C51" (id 0) (at 200.66 53.3399 0)
       (effects (font (size 1.27 1.27)) (justify left))
     )
@@
   (symbol (lib_id "power:GND") (at 109.22 151.13 0) (unit 1)
     (in_bom yes) (on_board yes) (fields_autoplaced)
-    (property "Reference" "#PWR?" (id 0) (at 109.22 157.48 0)
+    (property "Reference" "#PWR055" (id 0) (at 109.22 157.48 0)
       (effects (font (size 1.27 1.27)) hide)
     )
@@
   (symbol (lib_id "power:GND") (at 181.61 62.23 0) (unit 1)
     (in_bom yes) (on_board yes) (fields_autoplaced)
-    (property "Reference" "#PWR?" (id 0) (at 181.61 68.58 0)
+    (property "Reference" "#PWR059" (id 0) (at 181.61 68.58 0)
       (effects (font (size 1.27 1.27)) hide)
     )
@@
   (symbol (lib_id "power:+5V") (at 196.85 48.26 0) (unit 1)
     (in_bom yes) (on_board yes) (fields_autoplaced)
-    (property "Reference" "#PWR?" (id 0) (at 196.85 52.07 0)
+    (property "Reference" "#PWR060" (id 0) (at 196.85 52.07 0)
       (effects (font (size 1.27 1.27)) hide)
     )
@@
   (symbol (lib_id "Regulator_Linear:MC78L05_TO92") (at 181.61 50.8 0) (unit 1)
     (in_bom yes) (on_board yes) (fields_autoplaced)
-    (property "Reference" "U?" (id 0) (at 181.61 43.18 0))
+    (property "Reference" "U8" (id 0) (at 181.61 43.18 0))
     (property "Value" "" (id 1) (at 181.61 45.72 0))
     (property "Footprint" "" (id 2) (at 181.61 45.085 0)
@@
   (symbol (lib_id "power:GND") (at 133.35 151.13 0) (unit 1)
     (in_bom yes) (on_board yes) (fields_autoplaced)
-    (property "Reference" "#PWR?" (id 0) (at 133.35 157.48 0)
+    (property "Reference" "#PWR056" (id 0) (at 133.35 157.48 0)
       (effects (font (size 1.27 1.27)) hide)
     )
@@
   (symbol (lib_id "Device:R") (at 91.44 138.43 90) (unit 1)
     (in_bom yes) (on_board yes) (fields_autoplaced)
-    (property "Reference" "R?" (id 0) (at 91.44 132.08 90))
+    (property "Reference" "R73" (id 0) (at 91.44 132.08 90))
     (property "Value" "" (id 1) (at 91.44 134.62 90))
     (property "Footprint" "" (id 2) (at 91.44 140.208 90)
@@
   (symbol (lib_id "Device:R") (at 146.05 125.73 90) (unit 1)
     (in_bom yes) (on_board yes) (fields_autoplaced)
-    (property "Reference" "R?" (id 0) (at 146.05 119.38 90))
+    (property "Reference" "R74" (id 0) (at 146.05 119.38 90))
     (property "Value" "102k" (id 1) (at 146.05 121.92 90))
     (property "Footprint" "Resistor_SMD:R_0603_1608Metric" (id 2) (at 146.05 127.508 90)
@@
   (symbol (lib_id "power:+9V") (at 162.56 48.26 0) (unit 1)
     (in_bom yes) (on_board yes) (fields_autoplaced)
-    (property "Reference" "#PWR?" (id 0) (at 162.56 52.07 0)
+    (property "Reference" "#PWR058" (id 0) (at 162.56 52.07 0)
       (effects (font (size 1.27 1.27)) hide)
     )
@@
   (symbol (lib_id "Device:C_Polarized") (at 133.35 146.05 0) (unit 1)
     (in_bom yes) (on_board yes) (fields_autoplaced)
-    (property "Reference" "C?" (id 0) (at 137.16 143.8909 0)
+    (property "Reference" "C55" (id 0) (at 137.16 143.8909 0)
       (effects (font (size 1.27 1.27)) (justify left))
     )
@@
   (symbol (lib_id "power:-5V") (at 156.21 123.19 0) (unit 1)
     (in_bom yes) (on_board yes) (fields_autoplaced)
-    (property "Reference" "#PWR?" (id 0) (at 156.21 120.65 0)
+    (property "Reference" "#PWR057" (id 0) (at 156.21 120.65 0)
       (effects (font (size 1.27 1.27)) hide)
     )
@@
   (symbol (lib_id "Device:C") (at 73.66 132.08 0) (unit 1)
     (in_bom yes) (on_board yes) (fields_autoplaced)
-    (property "Reference" "C?" (id 0) (at 77.47 130.8099 0)
-      (effects (font (size 1.27 1.27)) (justify left))
-    )
+    (property "Reference" "C53" (id 0) (at 77.47 130.8099 0)
+      (effects (font (size 1.27 1.27)) (justify left))
+    )

Commit message: Sourced on_off switch and added on_off switch/indicator circuit
Parts:
- added D71: (no value), symbol User_Global_Symbol_Library:LED
- added R82: (no value), symbol Device:R
- added SW2: (no value), symbol Switch:SW_SPST
- C50: value (none) -> 0.33uF; footprint (none) -> Capacitor_SMD:C_0603_1608Metric
- C51: value (none) -> 0.1uF; footprint (none) -> Capacitor_SMD:C_0805_2012Metric
- C53: value (none) -> 1u; footprint (none) -> Capacitor_SMD:C_0402_1005Metric
- C54: value (none) -> 10u; footprint (none) -> Capacitor_SMD:C_0805_2012Metric
- C55: value (none) -> 100u; footprint (none) -> Capacitor_THT:C_Radial_D5.0mm_H5.0mm_P2.00mm
- C56: value (none) -> 0.002u; footprint (none) -> Capacitor_SMD:C_0402_1005Metric
- J2: value (none) -> PJ-070BH-SMT-TR; footprint (none) -> DC_Power_Jack_PJ_070BH_SMT_TR:CUI_PJ-PJ-070BH-SMT-TR
- R73: value (none) -> 20k; footprint (none) -> Resistor_SMD:R_0603_1608Metric
- U7: value (none) -> LT1054; footprint (none) -> LT1054_PDIP_Lin_Reg:DIP794W45P254L959H508Q8
- U8: value (none) -> MC78L05_TO92; footprint (none) -> Package_TO_SOT_THT:TO-92_Inline
Connections:
- net +9V: now also R82.1, SW2.2 (B); no longer J2.1
- net GND: now also D71.1 (K)
- new net: D71.2 (A), R82.2
- new net Power: J2.1, SW2.1 (A)
Other:
- moved on the sheet: J2

Commit message: Got 3D models for all parts, corrected signal voltage to each driver and made outline of PCB
Parts:
- removed J2: PJ-070BH-SMT-TR, DC_Power_Jack_PJ_070BH_SMT_TR:CUI_PJ-PJ-070BH-SMT-TR, symbol DC_Power_Jack _PJ_070BH_SMT_TR:PJ-070BH-SMT-TR
- added J2: (no value), symbol DC_Power_Jack _PJ_070BH:PJ-079BH
- D71: value (none) -> LED; footprint (none) -> LED_THT:LED_D5.0mm
- R82: value (none) -> 330; footprint (none) -> Resistor_SMD:R_0603_1608Metric
- SW2: value (none) -> SW_SPST; footprint (none) -> PW_On_Off_Switch:E-SWITCH_RR511D1121
Connections:
- net GND: now also J2.2, J2.3
- net Power: now also J2.1
- new net: J2.S1 (SHIELD), J2.S2 (SHIELD)
Changed lines of the file:
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@@
+    (stroke (width 0) (type default) (color 0 0 0 0))
+  )
+  (wire (pts (xy 64.77 55.88) (xy 64.77 52.07))
     (stroke (width 0) (type default) (color 0 0 0 0))
   )
@@
     (in_bom yes) (on_board yes) (fields_autoplaced)
     (property "Reference" "SW2" (id 0) (at 59.69 45.72 0))
-    (property "Value" "" (id 1) (at 59.69 48.26 0))
-    (property "Footprint" "" (id 2) (at 59.69 52.07 0)
+    (property "Value" "SW_SPST" (id 1) (at 59.69 48.26 0))
+    (property "Footprint" "PW_On_Off_Switch:E-SWITCH_RR511D1121" (id 2) (at 59.69 52.07 0)
       (effects (font (size 1.27 1.27)) hide)
     )
@@
     (pin "1")
     (pin "2")
+  )
+  (symbol (lib_id "power:PWR_FLAG") (at 156.21 125.73 270) (unit 1)
+    (in_bom yes) (on_board yes) (fields_autoplaced)
+    (property "Reference" "#FLG02" (id 0) (at 158.115 125.73 0)
+      (effects (font (size 1.27 1.27)) hide)
+    )
+    (property "Value" "PWR_FLAG" (id 1) (at 160.02 125.7299 90)
+      (effects (font (size 1.27 1.27)) (justify left))
+    )
+    (property "Footprint" "" (id 2) (at 156.21 125.73 0)
+      (effects (font (size 1.27 1.27)) hide)
+    )
+    (property "Datasheet" "~" (id 3) (at 156.21 125.73 0)
+      (effects (font (size 1.27 1.27)) hide)
+    )
+    (pin "1")
   )
   (symbol (lib_id "Device:C") (at 146.05 138.43 90) (unit 1)
@@
     (in_bom yes) (on_board yes) (fields_autoplaced)
     (property "Reference" "R82" (id 0) (at 77.47 45.72 90))
-    (property "Value" "" (id 1) (at 77.47 48.26 90))
-    (property "Footprint" "" (id 2) (at 77.47 53.848 90)
+    (property "Value" "330" (id 1) (at 77.47 48.26 90))
+    (property "Footprint" "Resistor_SMD:R_0603_1608Metric" (id 2) (at 77.47 53.848 90)
       (effects (font (size 1.27 1.27)) hide)
     )
@@
       (effects (font (size 1.27 1.27)) (justify right))
     )
-    (property "Value" "" (id 1) (at 90.4874 48.26 90)
+    (property "Value" "LED" (id 1) (at 90.4874 48.26 90)
       (effects (font (size 1.27 1.27)) (justify right))
     )
-    (property "Footprint" "" (id 2) (at 87.63 52.07 0)
+    (property "Footprint" "LED_THT:LED_D5.0mm" (id 2) (at 87.63 52.07 0)
       (effects (font (size 1.27 1.27)) hide)
     )
@@
     (pin "1")
   )
+  (symbol (lib_id "power:PWR_FLAG") (at 64.77 55.88 180) (unit 1)
+    (in_bom yes) (on_board yes) (fields_autoplaced)
+    (property "Reference" "#FLG01" (id 0) (at 64.77 57.785 0)
+      (effects (font (size 1.27 1.27)) hide)
+    )
+    (property "Value" "PWR_FLAG" (id 1) (at 64.77 60.96 0))
+    (property "Footprint" "" (id 2) (at 64.77 55.88 0)
+      (effects (font (size 1.27 1.27)) hide)
+    )
+    (property "Datasheet" "~" (id 3) (at 64.77 55.88 0)
+      (effects (font (size 1.27 1.27)) hide)
+    )
+    (pin "1")
+  )
   (symbol (lib_id "power:+5V") (at 196.85 48.26 0) (unit 1)
     (in_bom yes) (on_board yes) (fields_autoplaced)
@@
     (pin "3")
   )
-  (symbol (lib_id "DC_Power_Jack _PJ_070BH_SMT_TR:PJ-070BH-SMT-TR") (at 39.37 54.61 0) (unit 1)
-    (in_bom yes) (on_board yes) (fields_autoplaced)
-    (property "Reference" "J2" (id 0) (at 36.83 44.45 0))
-    (property "Value" "PJ-070BH-SMT-TR" (id 1) (at 36.83 46.99 0))
-    (property "Footprint" "DC_Power_Jack_PJ_070BH_SMT_TR:CUI_PJ-PJ-070BH-SMT-TR" (id 2) (at 39.37 54.61 0)
-      (effects (font (size 1.27 1.27)) (justify left bottom) hide)
-    )
-    (property "Datasheet" "" (id 3) (at 39.37 54.61 0)
-      (effects (font (size 1.27 1.27)) (justify left bottom) hide)
-    )
-    (property "MANUFACTURER" "CUI" (id 4) (at 39.37 54.61 0)
-      (effects (font (size 1.27 1.27)) (justify left bottom) hide)
-    )
-    (property "PARTREV" "1.05" (id 5) (at 39.37 54.61 0)
-      (effects (font (size 1.27 1.27)) (justify left bottom) hide)
-    )
-    (property "STANDARD" "Manufacturer Recommendations" (id 6) (at 39.37 54.61 0)
-      (effects (font (size 1.27 1.27)) (justify left bottom) hide)
-    )
-    (pin "1")
-    (pin "2")
-    (pin "3")
-  )
   (symbol (lib_id "power:GND") (at 133.35 151.13 0) (unit 1)
     (in_bom yes) (on_board yes) (fields_autoplaced)
@@
       (effects (font (size 1.27 1.27)) hide)
     )
-    (property "Value" "" (id 1) (at 101.6 52.07 0))
+    (property "Value" "GND" (id 1) (at 101.6 52.07 0))
     (property "Footprint" "" (id 2) (at 96.52 52.07 0)
       (effects (font (size 1.27 1.27)) hide)
@@
     (pin "1")
     (pin "2")
+  )
+  (symbol (lib_id "DC_Power_Jack _PJ_070BH:PJ-079BH") (at 31.75 57.15 0) (unit 1)
+    (in_bom yes) (on_board yes) (fields_autoplaced)
+    (property "Reference" "J2" (id 0) (at 31.75 44.45 0))
+    (property "Value" "" (id 1) (at 31.75 46.99 0))
+    (property "Footprint" "" (id 2) (at 31.75 57.15 0)
+      (effects (font (size 1.27 1.27)) (justify left bottom) hide)
+    )
+    (property "Datasheet" "" (id 3) (at 31.75 57.15 0)
+      (effects (font (size 1.27 1.27)) (justify left bottom) hide)
+    )
+    (property "MANUFACTURER" "CUI Inc" (id 4) (at 31.75 57.15 0)
+      (effects (font (size 1.27 1.27)) (justify left bottom) hide)
+    )
+    (property "PARTREV" "LTR" (id 5) (at 31.75 57.15 0)
+      (effects (font (size 1.27 1.27)) (justify left bottom) hide)
+    )
+    (property "STANDART" "Manufacturer Recommendations" (id 6) (at 31.75 57.15 0)
+      (effects (font (size 1.27 1.27)) (justify left bottom) hide)
+    )
+    (pin "1")
+    (pin "2")
+    (pin "3")
+    (pin "S1")
+    (pin "S2")
   )
   (symbol (lib_id "power:-5V") (at 156.21 123.19 0) (unit 1)
@@
       (effects (font (size 1.27 1.27)) hide)
     )
+    (pin "1")
+  )
+  (symbol (lib_id "power:PWR_FLAG") (at 196.85 50.8 270) (unit 1)
+    (in_bom yes) (on_board yes)
+    (property "Reference" "#FLG03" (id 0) (at 198.755 50.8 0)
+      (effects (font (size 1.27 1.27)) hide)
+    )
+    (property "Value" "PWR_FLAG" (id 1) (at 200.66 50.7999 90)
+      (effects (font (size 1.27 1.27)) (justify left))
+    )
+    (property "Footprint" "" (id 2) (at 196.85 50.8 0)
+      (effects (font (size 1.27 1.27)) hide)
+    )
+    (property "Datasheet" "~" (id 3) (at 196.85 50.8 0)
+      (effects (font (size 1.27 1.27)) hide)
+    )

Commit message: Both parts ar PVT09A 5K ohms, corrected footprint terminal labels
Parts:
- J2: value (none) -> PJ-079BH; footprint (none) -> CUI_PJ-079BH
Changed lines of the file:
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@@
     (in_bom yes) (on_board yes) (fields_autoplaced)
     (property "Reference" "J2" (id 0) (at 31.75 44.45 0))
-    (property "Value" "" (id 1) (at 31.75 46.99 0))
-    (property "Footprint" "" (id 2) (at 31.75 57.15 0)
+    (property "Value" "PJ-079BH" (id 1) (at 31.75 46.99 0))
+    (property "Footprint" "CUI_PJ-079BH" (id 2) (at 31.75 57.15 0)
       (effects (font (size 1.27 1.27)) (justify left bottom) hide)
     )

Commit message: Added 7th LM324 Quad-op-amp IC to Filter array, updated numbering on all other ICs
Parts:
- renumbered U7 to U8, U8 to U9
Changed lines of the file:
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@@
   (symbol (lib_id "Regulator_SwitchedCapacitor:LT1054") (at 109.22 133.35 0) (unit 1)
     (in_bom yes) (on_board yes) (fields_autoplaced)
-    (property "Reference" "U7" (id 0) (at 109.22 118.11 0))
+    (property "Reference" "U8" (id 0) (at 109.22 118.11 0))
     (property "Value" "LT1054" (id 1) (at 109.22 120.65 0))
     (property "Footprint" "LT1054_PDIP_Lin_Reg:DIP794W45P254L959H508Q8" (id 2) (at 111.76 135.89 0)
@@
   (symbol (lib_id "Regulator_Linear:MC78L05_TO92") (at 181.61 50.8 0) (unit 1)
     (in_bom yes) (on_board yes) (fields_autoplaced)
-    (property "Reference" "U8" (id 0) (at 181.61 43.18 0))
+    (property "Reference" "U9" (id 0) (at 181.61 43.18 0))
     (property "Value" "MC78L05_TO92" (id 1) (at 181.61 45.72 0))
     (property "Footprint" "Package_TO_SOT_THT:TO-92_Inline" (id 2) (at 181.61 45.085 0)
