File: Schematic_PCB/Music_Visualizer/Power.kicad_sch (KiCad schematic)
At the start: 16 parts, among them J2 PJ-079BH, Q1 DMP2123LQ-7, SW2 SW_SPST, U8 LT1054, U9 MC78L05_TO92

Commit message: Changed 0603 footprint to hand solder version, and changed 0402 footprints to 0603 hand solder version
Parts:
- C50: value 0.33uF -> (none); footprint Capacitor_SMD:C_0603_1608Metric -> (none)
- C52, C53: value 1u -> (none); footprint Capacitor_SMD:C_0402_1005Metric -> (none)
- C56: value 0.002u -> (none); footprint Capacitor_SMD:C_0402_1005Metric -> (none)
- R74: value 102k -> (none); footprint Resistor_SMD:R_0603_1608Metric -> (none)
- R82: value 330 -> (none); footprint Resistor_SMD:R_0603_1608Metric -> (none)
Changed lines of the file:
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@@
       (effects (font (size 1.27 1.27)) (justify left))
     )
-    (property "Value" "1u" (id 1) (at 64.77 133.3499 0)
-      (effects (font (size 1.27 1.27)) (justify left))
-    )
-    (property "Footprint" "Capacitor_SMD:C_0402_1005Metric" (id 2) (at 61.9252 135.89 0)
+    (property "Value" "" (id 1) (at 64.77 133.3499 0)
+      (effects (font (size 1.27 1.27)) (justify left))
+    )
+    (property "Footprint" "" (id 2) (at 61.9252 135.89 0)
       (effects (font (size 1.27 1.27)) hide)
     )
@@
       (effects (font (size 1.27 1.27)) (justify left))
     )
-    (property "Value" "0.33uF" (id 1) (at 166.37 55.8799 0)
-      (effects (font (size 1.27 1.27)) (justify left))
-    )
-    (property "Footprint" "Capacitor_SMD:C_0603_1608Metric" (id 2) (at 163.5252 58.42 0)
+    (property "Value" "" (id 1) (at 166.37 55.8799 0)
+      (effects (font (size 1.27 1.27)) (justify left))
+    )
+    (property "Footprint" "" (id 2) (at 163.5252 58.42 0)
       (effects (font (size 1.27 1.27)) hide)
     )
@@
     (in_bom yes) (on_board yes) (fields_autoplaced)
     (property "Reference" "C56" (id 0) (at 152.4 130.81 90))
-    (property "Value" "0.002u" (id 1) (at 152.4 133.35 90))
-    (property "Footprint" "Capacitor_SMD:C_0402_1005Metric" (id 2) (at 156.21 137.4648 0)
+    (property "Value" "" (id 1) (at 152.4 133.35 90))
+    (property "Footprint" "" (id 2) (at 156.21 137.4648 0)
       (effects (font (size 1.27 1.27)) hide)
     )
@@
     (in_bom yes) (on_board yes) (fields_autoplaced)
     (property "Reference" "R82" (id 0) (at 91.44 58.42 90))
-    (property "Value" "330" (id 1) (at 88.9 58.42 90))
-    (property "Footprint" "Resistor_SMD:R_0603_1608Metric" (id 2) (at 83.312 58.42 90)
+    (property "Value" "" (id 1) (at 88.9 58.42 90))
+    (property "Footprint" "" (id 2) (at 83.312 58.42 90)
       (effects (font (size 1.27 1.27)) hide)
     )
@@
     (in_bom yes) (on_board yes) (fields_autoplaced)
     (property "Reference" "R74" (id 0) (at 152.4 119.38 90))
-    (property "Value" "102k" (id 1) (at 152.4 121.92 90))
-    (property "Footprint" "Resistor_SMD:R_0603_1608Metric" (id 2) (at 152.4 127.508 90)
+    (property "Value" "" (id 1) (at 152.4 121.92 90))
+    (property "Footprint" "" (id 2) (at 152.4 127.508 90)
       (effects (font (size 1.27 1.27)) hide)
     )
@@
       (effects (font (size 1.27 1.27)) (justify left))
     )
-    (property "Value" "1u" (id 1) (at 77.47 133.3499 0)
-      (effects (font (size 1.27 1.27)) (justify left))
-    )
-    (property "Footprint" "Capacitor_SMD:C_0402_1005Metric" (id 2) (at 74.6252 135.89 0)
-      (effects (font (size 1.27 1.27)) hide)
-    )
+    (property "Value" "" (id 1) (at 77.47 133.3499 0)
+      (effects (font (size 1.27 1.27)) (justify left))
+    )
+    (property "Footprint" "" (id 2) (at 74.6252 135.89 0)
+      (effects (font (size 1.27 1.27)) hide)
+    )

Commit message: Corrected Resistor footprints from Capacitor_SMD to Resistor_SMD and created BOM
Parts:
- C50: value (none) -> 0.33uF; footprint (none) -> Capacitor_SMD:C_0603_1608Metric_Pad1.08x0.95mm_HandSolder
- C52, C53: value (none) -> 1u; footprint (none) -> Capacitor_SMD:C_0603_1608Metric_Pad1.08x0.95mm_HandSolder
- C56: value (none) -> 0.002u; footprint (none) -> Capacitor_SMD:C_0603_1608Metric_Pad1.08x0.95mm_HandSolder
- R73: value 20k -> (none); footprint Resistor_SMD:R_0603_1608Metric -> (none)
Changed lines of the file:
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@@
       (effects (font (size 1.27 1.27)) (justify left))
     )
-    (property "Value" "" (id 1) (at 64.77 133.3499 0)
-      (effects (font (size 1.27 1.27)) (justify left))
-    )
-    (property "Footprint" "" (id 2) (at 61.9252 135.89 0)
+    (property "Value" "1u" (id 1) (at 64.77 133.3499 0)
+      (effects (font (size 1.27 1.27)) (justify left))
+    )
+    (property "Footprint" "Capacitor_SMD:C_0603_1608Metric_Pad1.08x0.95mm_HandSolder" (id 2) (at 61.9252 135.89 0)
       (effects (font (size 1.27 1.27)) hide)
     )
@@
       (effects (font (size 1.27 1.27)) (justify left))
     )
-    (property "Value" "" (id 1) (at 166.37 55.8799 0)
-      (effects (font (size 1.27 1.27)) (justify left))
-    )
-    (property "Footprint" "" (id 2) (at 163.5252 58.42 0)
+    (property "Value" "0.33uF" (id 1) (at 166.37 55.8799 0)
+      (effects (font (size 1.27 1.27)) (justify left))
+    )
+    (property "Footprint" "Capacitor_SMD:C_0603_1608Metric_Pad1.08x0.95mm_HandSolder" (id 2) (at 163.5252 58.42 0)
       (effects (font (size 1.27 1.27)) hide)
     )
@@
     (in_bom yes) (on_board yes) (fields_autoplaced)
     (property "Reference" "C56" (id 0) (at 152.4 130.81 90))
-    (property "Value" "" (id 1) (at 152.4 133.35 90))
-    (property "Footprint" "" (id 2) (at 156.21 137.4648 0)
+    (property "Value" "0.002u" (id 1) (at 152.4 133.35 90))
+    (property "Footprint" "Capacitor_SMD:C_0603_1608Metric_Pad1.08x0.95mm_HandSolder" (id 2) (at 156.21 137.4648 0)
       (effects (font (size 1.27 1.27)) hide)
     )
@@
     (in_bom yes) (on_board yes) (fields_autoplaced)
     (property "Reference" "R73" (id 0) (at 88.9 132.08 90))
-    (property "Value" "20k" (id 1) (at 88.9 134.62 90))
-    (property "Footprint" "Resistor_SMD:R_0603_1608Metric" (id 2) (at 88.9 140.208 90)
+    (property "Value" "" (id 1) (at 88.9 134.62 90))
+    (property "Footprint" "" (id 2) (at 88.9 140.208 90)
       (effects (font (size 1.27 1.27)) hide)
     )
@@
       (effects (font (size 1.27 1.27)) (justify left))
     )
-    (property "Value" "" (id 1) (at 77.47 133.3499 0)
-      (effects (font (size 1.27 1.27)) (justify left))
-    )
-    (property "Footprint" "" (id 2) (at 74.6252 135.89 0)
-      (effects (font (size 1.27 1.27)) hide)
-    )
+    (property "Value" "1u" (id 1) (at 77.47 133.3499 0)
+      (effects (font (size 1.27 1.27)) (justify left))
+    )
+    (property "Footprint" "Capacitor_SMD:C_0603_1608Metric_Pad1.08x0.95mm_HandSolder" (id 2) (at 74.6252 135.89 0)
+      (effects (font (size 1.27 1.27)) hide)
+    )

Commit message: Corrected Spectrum Filter mistakes
In Kicad, op amp filters were connected as positive feedback, changed to negative feedback; corrected R5 and R8 values in FinalLowMidrange LTSpice file; corrected R2 and R3 in FinalUpperMidrange LTspice file; corrected R2 in FinalPresence LTSpice file; changed C39 and C40 in Kicad Brilliance Filter from 1nF to 820pF
Parts:
- R73: value (none) -> 20k; footprint (none) -> Resistor_SMD:R_0603_1608Metric_Pad0.98x0.95mm_HandSolder
- R74: value (none) -> 102k; footprint (none) -> Resistor_SMD:R_0603_1608Metric_Pad0.98x0.95mm_HandSolder
- R82: value (none) -> 330; footprint (none) -> Resistor_SMD:R_0603_1608Metric_Pad0.98x0.95mm_HandSolder
Changed lines of the file:
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@@
     (in_bom yes) (on_board yes) (fields_autoplaced)
     (property "Reference" "R82" (id 0) (at 91.44 58.42 90))
-    (property "Value" "" (id 1) (at 88.9 58.42 90))
-    (property "Footprint" "" (id 2) (at 83.312 58.42 90)
+    (property "Value" "330" (id 1) (at 88.9 58.42 90))
+    (property "Footprint" "Resistor_SMD:R_0603_1608Metric_Pad0.98x0.95mm_HandSolder" (id 2) (at 83.312 58.42 90)
       (effects (font (size 1.27 1.27)) hide)
     )
@@
     (in_bom yes) (on_board yes) (fields_autoplaced)
     (property "Reference" "R73" (id 0) (at 88.9 132.08 90))
-    (property "Value" "" (id 1) (at 88.9 134.62 90))
-    (property "Footprint" "" (id 2) (at 88.9 140.208 90)
+    (property "Value" "20k" (id 1) (at 88.9 134.62 90))
+    (property "Footprint" "Resistor_SMD:R_0603_1608Metric_Pad0.98x0.95mm_HandSolder" (id 2) (at 88.9 140.208 90)
       (effects (font (size 1.27 1.27)) hide)
     )
@@
     (in_bom yes) (on_board yes) (fields_autoplaced)
     (property "Reference" "R74" (id 0) (at 152.4 119.38 90))
-    (property "Value" "" (id 1) (at 152.4 121.92 90))
-    (property "Footprint" "" (id 2) (at 152.4 127.508 90)
+    (property "Value" "102k" (id 1) (at 152.4 121.92 90))
+    (property "Footprint" "Resistor_SMD:R_0603_1608Metric_Pad0.98x0.95mm_HandSolder" (id 2) (at 152.4 127.508 90)
       (effects (font (size 1.27 1.27)) hide)
     )

Commit message: Labeled output of U17 (3.5V LDO) 3.5V
Parts:
- R82: value 330 -> (none); footprint Resistor_SMD:R_0603_1608Metric_Pad0.98x0.95mm_HandSolder -> (none)
Changed lines of the file:
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@@
     (in_bom yes) (on_board yes) (fields_autoplaced)
     (property "Reference" "R82" (id 0) (at 91.44 58.42 90))
-    (property "Value" "330" (id 1) (at 88.9 58.42 90))
-    (property "Footprint" "Resistor_SMD:R_0603_1608Metric_Pad0.98x0.95mm_HandSolder" (id 2) (at 83.312 58.42 90)
+    (property "Value" "" (id 1) (at 88.9 58.42 90))
+    (property "Footprint" "" (id 2) (at 83.312 58.42 90)
       (effects (font (size 1.27 1.27)) hide)
     )
