File: Schematic_PCB/Music_Visualizer/Music_Visualizer.kicad_sch (KiCad schematic)
At the start: 145 parts, among them J1 AudioJack3, J3 Screw_Terminal_01x02, SW1 SW_SPDT, U1 LM324, U2 LM324, U3 LM324, U4 LM324, U5 LM324, U6 LM324, U7 LM324

Commit message: Corrected Resistor footprints from Capacitor_SMD to Resistor_SMD and created BOM
Parts:
- C19, C20: value (none) -> 1.6n; footprint (none) -> Capacitor_SMD:C_0603_1608Metric_Pad1.08x0.95mm_HandSolder
- C23, C24: value (none) -> 3n; footprint (none) -> Capacitor_SMD:C_0603_1608Metric_Pad1.08x0.95mm_HandSolder
- C4: value (none) -> 27n; footprint (none) -> Capacitor_SMD:C_0603_1608Metric_Pad1.08x0.95mm_HandSolder
- C47, C48, C49: value (none) -> 1u; footprint (none) -> Capacitor_SMD:C_0603_1608Metric_Pad1.08x0.95mm_HandSolder
- R1: value 84.5k -> (none); footprint Capacitor_SMD:C_0603_1608Metric_Pad1.08x0.95mm_HandSolder -> (none)
- R10: value 110k -> (none); footprint Capacitor_SMD:C_0603_1608Metric_Pad1.08x0.95mm_HandSolder -> (none)
- R11, R4, R65: value 90.9k -> (none); footprint Capacitor_SMD:C_0603_1608Metric_Pad1.08x0.95mm_HandSolder -> (none)
- R12: value 162k -> (none); footprint Capacitor_SMD:C_0603_1608Metric_Pad1.08x0.95mm_HandSolder -> (none)
- R13: value 118k -> (none); footprint Capacitor_SMD:C_0603_1608Metric_Pad1.08x0.95mm_HandSolder -> (none)
- R14: value 63.4k -> (none); footprint Capacitor_SMD:C_0603_1608Metric_Pad1.08x0.95mm_HandSolder -> (none)
- R15: value 62k -> (none); footprint Capacitor_SMD:C_0603_1608Metric_Pad1.08x0.95mm_HandSolder -> (none)
- R16: value 309k -> (none); footprint Capacitor_SMD:C_0603_1608Metric_Pad1.08x0.95mm_HandSolder -> (none)
- R17: value 68k -> (none); footprint Capacitor_SMD:C_0603_1608Metric_Pad1.08x0.95mm_HandSolder -> (none)
- R18, R31, R36, R51: value 66.5k -> (none); footprint Capacitor_SMD:C_0603_1608Metric_Pad1.08x0.95mm_HandSolder -> (none)
- R19: value 332k -> (none); footprint Capacitor_SMD:C_0603_1608Metric_Pad1.08x0.95mm_HandSolder -> (none)
- R2, R41, R50: value 160k -> (none); footprint Capacitor_SMD:C_0603_1608Metric_Pad1.08x0.95mm_HandSolder -> (none)
- R20: value 137k -> (none); footprint Capacitor_SMD:C_0603_1608Metric_Pad1.08x0.95mm_HandSolder -> (none)
- R21: value 45.3k -> (none); footprint Capacitor_SMD:C_0603_1608Metric_Pad1.08x0.95mm_HandSolder -> (none)
- R22, R35, R53: value 270k -> (none); footprint Capacitor_SMD:C_0603_1608Metric_Pad1.08x0.95mm_HandSolder -> (none)
- R23: value 143k -> (none); footprint Capacitor_SMD:C_0603_1608Metric_Pad1.08x0.95mm_HandSolder -> (none)
- R24: value 19.1k -> (none); footprint Capacitor_SMD:C_0603_1608Metric_Pad1.08x0.95mm_HandSolder -> (none)
- R25: value 590k -> (none); footprint Capacitor_SMD:C_0603_1608Metric_Pad1.08x0.95mm_HandSolder -> (none)
- R26: value 140k -> (none); footprint Capacitor_SMD:C_0603_1608Metric_Pad1.08x0.95mm_HandSolder -> (none)
- R27: value 18.7k -> (none); footprint Capacitor_SMD:C_0603_1608Metric_Pad1.08x0.95mm_HandSolder -> (none)
- R28: value 576k -> (none); footprint Capacitor_SMD:C_0603_1608Metric_Pad1.08x0.95mm_HandSolder -> (none)
- R29, R30: value 100k -> (none); footprint Capacitor_SMD:C_0603_1608Metric_Pad1.08x0.95mm_HandSolder -> (none)
- R3: value 169k -> (none); footprint Capacitor_SMD:C_0603_1608Metric_Pad1.08x0.95mm_HandSolder -> (none)
- R32: value 33.2k -> (none); footprint Capacitor_SMD:C_0603_1608Metric_Pad1.08x0.95mm_HandSolder -> (none)
- R33: value 56k -> (none); footprint Capacitor_SMD:C_0603_1608Metric_Pad1.08x0.95mm_HandSolder -> (none)
- R34, R58: value 48.7k -> (none); footprint Capacitor_SMD:C_0603_1608Metric_Pad1.08x0.95mm_HandSolder -> (none)
- R37: value 57.6k -> (none); footprint Capacitor_SMD:C_0603_1608Metric_Pad1.08x0.95mm_HandSolder -> (none)
- R38: value 324k -> (none); footprint Capacitor_SMD:C_0603_1608Metric_Pad1.08x0.95mm_HandSolder -> (none)
- R39, R48: value 78.7k -> (none); footprint Capacitor_SMD:C_0603_1608Metric_Pad1.08x0.95mm_HandSolder -> (none)
- R40: value 26.7k -> (none); footprint Capacitor_SMD:C_0603_1608Metric_Pad1.08x0.95mm_HandSolder -> (none)
- R42: value 59k -> (none); footprint Capacitor_SMD:C_0603_1608Metric_Pad1.08x0.95mm_HandSolder -> (none)
- R43: value 7.87k -> (none); footprint Capacitor_SMD:C_0603_1608Metric_Pad1.08x0.95mm_HandSolder -> (none)
- R44: value 243k -> (none); footprint Capacitor_SMD:C_0603_1608Metric_Pad1.08x0.95mm_HandSolder -> (none)
- R45: value 107k -> (none); footprint Capacitor_SMD:C_0603_1608Metric_Pad1.08x0.95mm_HandSolder -> (none)
- R46: value 14.7k -> (none); footprint Capacitor_SMD:C_0603_1608Metric_Pad1.08x0.95mm_HandSolder -> (none)
- R47: value 453k -> (none); footprint Capacitor_SMD:C_0603_1608Metric_Pad1.08x0.95mm_HandSolder -> (none)
- R49: value 7.32k -> (none); footprint Capacitor_SMD:C_0603_1608Metric_Pad1.08x0.95mm_HandSolder -> (none)
- R5, R62: value 37.4k -> (none); footprint Capacitor_SMD:C_0603_1608Metric_Pad1.08x0.95mm_HandSolder -> (none)
- R52: value 2.87k -> (none); footprint Capacitor_SMD:C_0603_1608Metric_Pad1.08x0.95mm_HandSolder -> (none)
- R54: value 95.3k -> (none); footprint Capacitor_SMD:C_0603_1608Metric_Pad1.08x0.95mm_HandSolder -> (none)
- R55: value 4.02k -> (none); footprint Capacitor_SMD:C_0603_1608Metric_Pad1.08x0.95mm_HandSolder -> (none)
- R56: value 383k -> (none); footprint Capacitor_SMD:C_0603_1608Metric_Pad1.08x0.95mm_HandSolder -> (none)
- R59: value 22.6k -> (none); footprint Capacitor_SMD:C_0603_1608Metric_Pad1.08x0.95mm_HandSolder -> (none)
- R6: value 402k -> (none); footprint Capacitor_SMD:C_0603_1608Metric_Pad1.08x0.95mm_HandSolder -> (none)
- R60: value 8.06k -> (none); footprint Capacitor_SMD:C_0603_1608Metric_Pad1.08x0.95mm_HandSolder -> (none)
- R61: value 4.32k -> (none); footprint Capacitor_SMD:C_0603_1608Metric_Pad1.08x0.95mm_HandSolder -> (none)
- R63: value 19.6k -> (none); footprint Capacitor_SMD:C_0603_1608Metric_Pad1.08x0.95mm_HandSolder -> (none)
- R64: value 10.7k -> (none); footprint Capacitor_SMD:C_0603_1608Metric_Pad1.08x0.95mm_HandSolder -> (none)
- R66, R67, R68, R69, R70, R71, R72: value 1k -> (none); footprint Capacitor_SMD:C_0603_1608Metric_Pad1.08x0.95mm_HandSolder -> (none)
- R7: value 86.6k -> (none); footprint Capacitor_SMD:C_0603_1608Metric_Pad1.08x0.95mm_HandSolder -> (none)
- R8: value 35.7k -> (none); footprint Capacitor_SMD:C_0603_1608Metric_Pad1.08x0.95mm_HandSolder -> (none)
- R9: value 390k -> (none); footprint Capacitor_SMD:C_0603_1608Metric_Pad1.08x0.95mm_HandSolder -> (none)

Commit message: Corrected Spectrum Filter mistakes
In Kicad, op amp filters were connected as positive feedback, changed to negative feedback; corrected R5 and R8 values in FinalLowMidrange LTSpice file; corrected R2 and R3 in FinalUpperMidrange LTspice file; corrected R2 in FinalPresence LTSpice file; changed C39 and C40 in Kicad Brilliance Filter from 1nF to 820pF
Parts:
- C39, C40: value 1n -> (none); footprint Capacitor_SMD:C_0603_1608Metric_Pad1.08x0.95mm_HandSolder -> (none)
- R1: value (none) -> 84.5k; footprint (none) -> Resistor_SMD:R_0603_1608Metric_Pad0.98x0.95mm_HandSolder
- R10: value (none) -> 110k; footprint (none) -> Resistor_SMD:R_0603_1608Metric_Pad0.98x0.95mm_HandSolder
- R11, R4, R65: value (none) -> 90.9k; footprint (none) -> Resistor_SMD:R_0603_1608Metric_Pad0.98x0.95mm_HandSolder
- R12: value (none) -> 162k; footprint (none) -> Resistor_SMD:R_0603_1608Metric_Pad0.98x0.95mm_HandSolder
- R13: value (none) -> 118k; footprint (none) -> Resistor_SMD:R_0603_1608Metric_Pad0.98x0.95mm_HandSolder
- R14: value (none) -> 63.4k; footprint (none) -> Resistor_SMD:R_0603_1608Metric_Pad0.98x0.95mm_HandSolder
- R15: value (none) -> 62k; footprint (none) -> Resistor_SMD:R_0603_1608Metric_Pad0.98x0.95mm_HandSolder
- R16: value (none) -> 309k; footprint (none) -> Resistor_SMD:R_0603_1608Metric_Pad0.98x0.95mm_HandSolder
- R17: value (none) -> 68k; footprint (none) -> Resistor_SMD:R_0603_1608Metric_Pad0.98x0.95mm_HandSolder
- R18, R31, R36, R51: value (none) -> 66.5k; footprint (none) -> Resistor_SMD:R_0603_1608Metric_Pad0.98x0.95mm_HandSolder
- R19: value (none) -> 332k; footprint (none) -> Resistor_SMD:R_0603_1608Metric_Pad0.98x0.95mm_HandSolder
- R2, R41, R50: value (none) -> 160k; footprint (none) -> Resistor_SMD:R_0603_1608Metric_Pad0.98x0.95mm_HandSolder
- R20: value (none) -> 137k; footprint (none) -> Resistor_SMD:R_0603_1608Metric_Pad0.98x0.95mm_HandSolder
- R21: value (none) -> 45.3k; footprint (none) -> Resistor_SMD:R_0603_1608Metric_Pad0.98x0.95mm_HandSolder
- R22, R35, R53: value (none) -> 270k; footprint (none) -> Resistor_SMD:R_0603_1608Metric_Pad0.98x0.95mm_HandSolder
- R23: value (none) -> 143k; footprint (none) -> Resistor_SMD:R_0603_1608Metric_Pad0.98x0.95mm_HandSolder
- R24: value (none) -> 19.1k; footprint (none) -> Resistor_SMD:R_0603_1608Metric_Pad0.98x0.95mm_HandSolder
- R25: value (none) -> 590k; footprint (none) -> Resistor_SMD:R_0603_1608Metric_Pad0.98x0.95mm_HandSolder
- R26: value (none) -> 140k; footprint (none) -> Resistor_SMD:R_0603_1608Metric_Pad0.98x0.95mm_HandSolder
- R27: value (none) -> 18.7k; footprint (none) -> Resistor_SMD:R_0603_1608Metric_Pad0.98x0.95mm_HandSolder
- R28: value (none) -> 576k; footprint (none) -> Resistor_SMD:R_0603_1608Metric_Pad0.98x0.95mm_HandSolder
- R29, R30: value (none) -> 100k; footprint (none) -> Resistor_SMD:R_0603_1608Metric_Pad0.98x0.95mm_HandSolder
- R3: value (none) -> 169k; footprint (none) -> Resistor_SMD:R_0603_1608Metric_Pad0.98x0.95mm_HandSolder
- R32: value (none) -> 33.2k; footprint (none) -> Resistor_SMD:R_0603_1608Metric_Pad0.98x0.95mm_HandSolder
- R33: value (none) -> 56k; footprint (none) -> Resistor_SMD:R_0603_1608Metric_Pad0.98x0.95mm_HandSolder
- R34, R58: value (none) -> 48.7k; footprint (none) -> Resistor_SMD:R_0603_1608Metric_Pad0.98x0.95mm_HandSolder
- R37: value (none) -> 57.6k; footprint (none) -> Resistor_SMD:R_0603_1608Metric_Pad0.98x0.95mm_HandSolder
- R38: value (none) -> 324k; footprint (none) -> Resistor_SMD:R_0603_1608Metric_Pad0.98x0.95mm_HandSolder
- R39, R48: value (none) -> 78.7k; footprint (none) -> Resistor_SMD:R_0603_1608Metric_Pad0.98x0.95mm_HandSolder
- R40: value (none) -> 26.7k; footprint (none) -> Resistor_SMD:R_0603_1608Metric_Pad0.98x0.95mm_HandSolder
- R42: value (none) -> 59k; footprint (none) -> Resistor_SMD:R_0603_1608Metric_Pad0.98x0.95mm_HandSolder
- R43: value (none) -> 7.87k; footprint (none) -> Resistor_SMD:R_0603_1608Metric_Pad0.98x0.95mm_HandSolder
- R44: value (none) -> 243k; footprint (none) -> Resistor_SMD:R_0603_1608Metric_Pad0.98x0.95mm_HandSolder
- R45: value (none) -> 107k; footprint (none) -> Resistor_SMD:R_0603_1608Metric_Pad0.98x0.95mm_HandSolder
- R46: value (none) -> 14.7k; footprint (none) -> Resistor_SMD:R_0603_1608Metric_Pad0.98x0.95mm_HandSolder
- R47: value (none) -> 453k; footprint (none) -> Resistor_SMD:R_0603_1608Metric_Pad0.98x0.95mm_HandSolder
- R49: value (none) -> 7.32k; footprint (none) -> Resistor_SMD:R_0603_1608Metric_Pad0.98x0.95mm_HandSolder
- R5, R62: value (none) -> 37.4k; footprint (none) -> Resistor_SMD:R_0603_1608Metric_Pad0.98x0.95mm_HandSolder
- R52: value (none) -> 2.87k; footprint (none) -> Resistor_SMD:R_0603_1608Metric_Pad0.98x0.95mm_HandSolder
- R54: value (none) -> 95.3k; footprint (none) -> Resistor_SMD:R_0603_1608Metric_Pad0.98x0.95mm_HandSolder
- R55: value (none) -> 4.02k; footprint (none) -> Resistor_SMD:R_0603_1608Metric_Pad0.98x0.95mm_HandSolder
- R56: value (none) -> 383k; footprint (none) -> Resistor_SMD:R_0603_1608Metric_Pad0.98x0.95mm_HandSolder
- R59: value (none) -> 22.6k; footprint (none) -> Resistor_SMD:R_0603_1608Metric_Pad0.98x0.95mm_HandSolder
- R6: value (none) -> 402k; footprint (none) -> Resistor_SMD:R_0603_1608Metric_Pad0.98x0.95mm_HandSolder
- R60: value (none) -> 8.06k; footprint (none) -> Resistor_SMD:R_0603_1608Metric_Pad0.98x0.95mm_HandSolder
- R61: value (none) -> 4.32k; footprint (none) -> Resistor_SMD:R_0603_1608Metric_Pad0.98x0.95mm_HandSolder
- R63: value (none) -> 19.6k; footprint (none) -> Resistor_SMD:R_0603_1608Metric_Pad0.98x0.95mm_HandSolder
- R64: value (none) -> 10.7k; footprint (none) -> Resistor_SMD:R_0603_1608Metric_Pad0.98x0.95mm_HandSolder
- R66, R67, R68, R69, R70, R71, R72: value (none) -> 1k; footprint (none) -> Resistor_SMD:R_0603_1608Metric_Pad0.98x0.95mm_HandSolder
- R7: value (none) -> 86.6k; footprint (none) -> Resistor_SMD:R_0603_1608Metric_Pad0.98x0.95mm_HandSolder
- R8: value (none) -> 35.7k; footprint (none) -> Resistor_SMD:R_0603_1608Metric_Pad0.98x0.95mm_HandSolder
- R9: value (none) -> 390k; footprint (none) -> Resistor_SMD:R_0603_1608Metric_Pad0.98x0.95mm_HandSolder
Connections:
- net GND: now also U1.10 (+), U1.3 (+), U1.5 (+), U2.10 (+), U2.5 (+), U3.10 (+), U3.3 (+), U3.5 (+), U4.10 (+), U4.5 (+), U5.10 (+), U5.3 (+), U5.5 (+), U6.10 (+), U6.3 (+), U6.5 (+), U7.10 (+), U7.3 (+), U7.5 (+); no longer U1.2 (-), U1.6 (-), U1.9 (-), U2.6 (-), U2.9 (-), U3.2 (-), U3.6 (-), U3.9 (-), U4.6 (-), U4.9 (-), U5.2 (-), U5.6 (-), U5.9 (-), U6.2 (-), U6.6 (-), U6.9 (-), U7.2 (-), U7.6 (-), U7.9 (-)
- net at C30.2, R47.2: now also U5.9 (-); no longer U5.10 (+)
- net at C36.2, R56.2: now also U6.9 (-); no longer U6.10 (+)
- net at C32.2, R50.2: now also U6.2 (-); no longer U6.3 (+)
- net at C16.2, R25.2: now also U3.6 (-); no longer U3.5 (+)
- net at C26.2, R41.2: now also U5.2 (-); no longer U5.3 (+)
- net at C38.2, R59.2: now also U7.2 (-); no longer U7.3 (+)
- net at C14.2, R22.2: now also U3.2 (-); no longer U3.3 (+)
- net at C2.2, R3.2: now also U1.2 (-); no longer U1.3 (+)
- net at C8.2, R11.2: now also U2.2 (-); no longer U2.3 (+)
- net at C12.2, R19.2: now also U2.9 (-); no longer U2.10 (+)
- net at C28.2, R44.2: now also U5.6 (-); no longer U5.5 (+)
- net at R31.2, R32.1: now also U4.3 (+); no longer U4.2 (-)
- net at C20.2, R30.2: now also U4.2 (-); no longer U4.3 (+)
- net at C4.2, R6.2: now also U1.6 (-); no longer U1.5 (+)
- net at R12.2, R13.1: now also U2.3 (+); no longer U2.2 (-)
- net at C42.2, R65.2: now also U7.9 (-); no longer U7.10 (+)
- net at C24.2, R38.2: now also U4.9 (-); no longer U4.10 (+)
- net at C10.2, R16.2: now also U2.6 (-); no longer U2.5 (+)
- net at C40.2, R62.2: now also U7.6 (-); no longer U7.5 (+)
- net at C6.2, R9.2: now also U1.9 (-); no longer U1.10 (+)
- net at C18.2, R28.2: now also U3.9 (-); no longer U3.10 (+)
- net at C34.2, R53.2: now also U6.6 (-); no longer U6.5 (+)
- net at C22.2, R35.2: now also U4.6 (-); no longer U4.5 (+)
