File: Schematic_PCB/Music_Visualizer/Led_Driver.kicad_sch (KiCad schematic)
At the start: 92 parts, among them U10 LM3915N-1, U11 LM3915N-1, U12 LM3915N-1, U13 LM3915N-1, U14 LM3915N-1, U15 LM3915N-1, U16 LM3915N-1, U17 NCP161ASN350T1G, U18 NCS333ASQ3T2G

Commit message: Changed 0603 footprint to hand solder version, and changed 0402 footprints to 0603 hand solder version
Parts:
- C57, C58: value 1u -> (none); footprint Capacitor_SMD:C_0402_1005Metric -> (none)
- R75, R76, R77, R78, R79, R80, R81: value 680 -> (none); footprint Resistor_SMD:R_0603_1608Metric -> (none)
Changed lines of the file:
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@@
       (effects (font (size 1.27 1.27)) (justify left))
     )
-    (property "Value" "680" (id 1) (at 82.55 255.2699 0)
-      (effects (font (size 1.27 1.27)) (justify left))
-    )
-    (property "Footprint" "Resistor_SMD:R_0603_1608Metric" (id 2) (at 78.232 254 90)
+    (property "Value" "" (id 1) (at 82.55 255.2699 0)
+      (effects (font (size 1.27 1.27)) (justify left))
+    )
+    (property "Footprint" "" (id 2) (at 78.232 254 90)
       (effects (font (size 1.27 1.27)) hide)
     )
@@
       (effects (font (size 1.27 1.27)) (justify left))
     )
-    (property "Value" "680" (id 1) (at 91.44 124.4599 0)
-      (effects (font (size 1.27 1.27)) (justify left))
-    )
-    (property "Footprint" "Resistor_SMD:R_0603_1608Metric" (id 2) (at 87.122 123.19 90)
+    (property "Value" "" (id 1) (at 91.44 124.4599 0)
+      (effects (font (size 1.27 1.27)) (justify left))
+    )
+    (property "Footprint" "" (id 2) (at 87.122 123.19 90)
       (effects (font (size 1.27 1.27)) hide)
     )
@@
       (effects (font (size 1.27 1.27)) (justify left))
     )
-    (property "Value" "680" (id 1) (at 255.27 372.1099 0)
-      (effects (font (size 1.27 1.27)) (justify left))
-    )
-    (property "Footprint" "Resistor_SMD:R_0603_1608Metric" (id 2) (at 250.952 370.84 90)
+    (property "Value" "" (id 1) (at 255.27 372.1099 0)
+      (effects (font (size 1.27 1.27)) (justify left))
+    )
+    (property "Footprint" "" (id 2) (at 250.952 370.84 90)
       (effects (font (size 1.27 1.27)) hide)
     )
@@
       (effects (font (size 1.27 1.27)) (justify left))
     )
-    (property "Value" "1u" (id 1) (at 440.69 223.5199 0)
-      (effects (font (size 1.27 1.27)) (justify left))
-    )
-    (property "Footprint" "Capacitor_SMD:C_0402_1005Metric" (id 2) (at 437.8452 226.06 0)
+    (property "Value" "" (id 1) (at 440.69 223.5199 0)
+      (effects (font (size 1.27 1.27)) (justify left))
+    )
+    (property "Footprint" "" (id 2) (at 437.8452 226.06 0)
       (effects (font (size 1.27 1.27)) hide)
     )
@@
       (effects (font (size 1.27 1.27)) (justify left))
     )
-    (property "Value" "680" (id 1) (at 83.82 370.8399 0)
-      (effects (font (size 1.27 1.27)) (justify left))
-    )
-    (property "Footprint" "Resistor_SMD:R_0603_1608Metric" (id 2) (at 79.502 369.57 90)
+    (property "Value" "" (id 1) (at 83.82 370.8399 0)
+      (effects (font (size 1.27 1.27)) (justify left))
+    )
+    (property "Footprint" "" (id 2) (at 79.502 369.57 90)
       (effects (font (size 1.27 1.27)) hide)
     )
@@
       (effects (font (size 1.27 1.27)) (justify left))
     )
-    (property "Value" "680" (id 1) (at 436.88 370.8399 0)
-      (effects (font (size 1.27 1.27)) (justify left))
-    )
-    (property "Footprint" "Resistor_SMD:R_0603_1608Metric" (id 2) (at 432.562 369.57 90)
+    (property "Value" "" (id 1) (at 436.88 370.8399 0)
+      (effects (font (size 1.27 1.27)) (justify left))
+    )
+    (property "Footprint" "" (id 2) (at 432.562 369.57 90)
       (effects (font (size 1.27 1.27)) hide)
     )
@@
       (effects (font (size 1.27 1.27)) (justify left))
     )
-    (property "Value" "680" (id 1) (at 254 123.1899 0)
-      (effects (font (size 1.27 1.27)) (justify left))
-    )
-    (property "Footprint" "Resistor_SMD:R_0603_1608Metric" (id 2) (at 249.682 121.92 90)
+    (property "Value" "" (id 1) (at 254 123.1899 0)
+      (effects (font (size 1.27 1.27)) (justify left))
+    )
+    (property "Footprint" "" (id 2) (at 249.682 121.92 90)
       (effects (font (size 1.27 1.27)) hide)
     )
@@
       (effects (font (size 1.27 1.27)) (justify left))
     )
-    (property "Value" "1u" (id 1) (at 472.44 223.5199 0)
-      (effects (font (size 1.27 1.27)) (justify left))
-    )
-    (property "Footprint" "Capacitor_SMD:C_0402_1005Metric" (id 2) (at 469.5952 226.06 0)
+    (property "Value" "" (id 1) (at 472.44 223.5199 0)
+      (effects (font (size 1.27 1.27)) (justify left))
+    )
+    (property "Footprint" "" (id 2) (at 469.5952 226.06 0)
       (effects (font (size 1.27 1.27)) hide)
     )
@@
       (effects (font (size 1.27 1.27)) (justify left))
     )
-    (property "Value" "680" (id 1) (at 427.99 123.1899 0)
-      (effects (font (size 1.27 1.27)) (justify left))
-    )
-    (property "Footprint" "Resistor_SMD:R_0603_1608Metric" (id 2) (at 423.672 121.92 90)
-      (effects (font (size 1.27 1.27)) hide)
-    )
+    (property "Value" "" (id 1) (at 427.99 123.1899 0)
+      (effects (font (size 1.27 1.27)) (justify left))
+    )
+    (property "Footprint" "" (id 2) (at 423.672 121.92 90)
+      (effects (font (size 1.27 1.27)) hide)
+    )

Commit message: Corrected Resistor footprints from Capacitor_SMD to Resistor_SMD and created BOM
Parts:
- C57, C58: value (none) -> 1u; footprint (none) -> Capacitor_SMD:C_0603_1608Metric_Pad1.08x0.95mm_HandSolder
Changed lines of the file:
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@@
       (effects (font (size 1.27 1.27)) (justify left))
     )
-    (property "Value" "" (id 1) (at 440.69 223.5199 0)
-      (effects (font (size 1.27 1.27)) (justify left))
-    )
-    (property "Footprint" "" (id 2) (at 437.8452 226.06 0)
+    (property "Value" "1u" (id 1) (at 440.69 223.5199 0)
+      (effects (font (size 1.27 1.27)) (justify left))
+    )
+    (property "Footprint" "Capacitor_SMD:C_0603_1608Metric_Pad1.08x0.95mm_HandSolder" (id 2) (at 437.8452 226.06 0)
       (effects (font (size 1.27 1.27)) hide)
     )
@@
       (effects (font (size 1.27 1.27)) (justify left))
     )
-    (property "Value" "" (id 1) (at 472.44 223.5199 0)
-      (effects (font (size 1.27 1.27)) (justify left))
-    )
-    (property "Footprint" "" (id 2) (at 469.5952 226.06 0)
-      (effects (font (size 1.27 1.27)) hide)
-    )
+    (property "Value" "1u" (id 1) (at 472.44 223.5199 0)
+      (effects (font (size 1.27 1.27)) (justify left))
+    )
+    (property "Footprint" "Capacitor_SMD:C_0603_1608Metric_Pad1.08x0.95mm_HandSolder" (id 2) (at 469.5952 226.06 0)
+      (effects (font (size 1.27 1.27)) hide)
+    )

Commit message: Corrected Spectrum Filter mistakes
In Kicad, op amp filters were connected as positive feedback, changed to negative feedback; corrected R5 and R8 values in FinalLowMidrange LTSpice file; corrected R2 and R3 in FinalUpperMidrange LTspice file; corrected R2 in FinalPresence LTSpice file; changed C39 and C40 in Kicad Brilliance Filter from 1nF to 820pF
Parts:
- R75, R76, R77, R78, R79, R80, R81: value (none) -> 680; footprint (none) -> Resistor_SMD:R_0603_1608Metric_Pad0.98x0.95mm_HandSolder
Changed lines of the file:
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@@
       (effects (font (size 1.27 1.27)) (justify left))
     )
-    (property "Value" "" (id 1) (at 82.55 255.2699 0)
-      (effects (font (size 1.27 1.27)) (justify left))
-    )
-    (property "Footprint" "" (id 2) (at 78.232 254 90)
+    (property "Value" "680" (id 1) (at 82.55 255.2699 0)
+      (effects (font (size 1.27 1.27)) (justify left))
+    )
+    (property "Footprint" "Resistor_SMD:R_0603_1608Metric_Pad0.98x0.95mm_HandSolder" (id 2) (at 78.232 254 90)
       (effects (font (size 1.27 1.27)) hide)
     )
@@
       (effects (font (size 1.27 1.27)) (justify left))
     )
-    (property "Value" "" (id 1) (at 91.44 124.4599 0)
-      (effects (font (size 1.27 1.27)) (justify left))
-    )
-    (property "Footprint" "" (id 2) (at 87.122 123.19 90)
+    (property "Value" "680" (id 1) (at 91.44 124.4599 0)
+      (effects (font (size 1.27 1.27)) (justify left))
+    )
+    (property "Footprint" "Resistor_SMD:R_0603_1608Metric_Pad0.98x0.95mm_HandSolder" (id 2) (at 87.122 123.19 90)
       (effects (font (size 1.27 1.27)) hide)
     )
@@
       (effects (font (size 1.27 1.27)) (justify left))
     )
-    (property "Value" "" (id 1) (at 255.27 372.1099 0)
-      (effects (font (size 1.27 1.27)) (justify left))
-    )
-    (property "Footprint" "" (id 2) (at 250.952 370.84 90)
+    (property "Value" "680" (id 1) (at 255.27 372.1099 0)
+      (effects (font (size 1.27 1.27)) (justify left))
+    )
+    (property "Footprint" "Resistor_SMD:R_0603_1608Metric_Pad0.98x0.95mm_HandSolder" (id 2) (at 250.952 370.84 90)
       (effects (font (size 1.27 1.27)) hide)
     )
@@
       (effects (font (size 1.27 1.27)) (justify left))
     )
-    (property "Value" "" (id 1) (at 83.82 370.8399 0)
-      (effects (font (size 1.27 1.27)) (justify left))
-    )
-    (property "Footprint" "" (id 2) (at 79.502 369.57 90)
+    (property "Value" "680" (id 1) (at 83.82 370.8399 0)
+      (effects (font (size 1.27 1.27)) (justify left))
+    )
+    (property "Footprint" "Resistor_SMD:R_0603_1608Metric_Pad0.98x0.95mm_HandSolder" (id 2) (at 79.502 369.57 90)
       (effects (font (size 1.27 1.27)) hide)
     )
@@
       (effects (font (size 1.27 1.27)) (justify left))
     )
-    (property "Value" "" (id 1) (at 436.88 370.8399 0)
-      (effects (font (size 1.27 1.27)) (justify left))
-    )
-    (property "Footprint" "" (id 2) (at 432.562 369.57 90)
+    (property "Value" "680" (id 1) (at 436.88 370.8399 0)
+      (effects (font (size 1.27 1.27)) (justify left))
+    )
+    (property "Footprint" "Resistor_SMD:R_0603_1608Metric_Pad0.98x0.95mm_HandSolder" (id 2) (at 432.562 369.57 90)
       (effects (font (size 1.27 1.27)) hide)
     )
@@
       (effects (font (size 1.27 1.27)) (justify left))
     )
-    (property "Value" "" (id 1) (at 254 123.1899 0)
-      (effects (font (size 1.27 1.27)) (justify left))
-    )
-    (property "Footprint" "" (id 2) (at 249.682 121.92 90)
+    (property "Value" "680" (id 1) (at 254 123.1899 0)
+      (effects (font (size 1.27 1.27)) (justify left))
+    )
+    (property "Footprint" "Resistor_SMD:R_0603_1608Metric_Pad0.98x0.95mm_HandSolder" (id 2) (at 249.682 121.92 90)
       (effects (font (size 1.27 1.27)) hide)
     )
@@
       (effects (font (size 1.27 1.27)) (justify left))
     )
-    (property "Value" "" (id 1) (at 427.99 123.1899 0)
-      (effects (font (size 1.27 1.27)) (justify left))
-    )
-    (property "Footprint" "" (id 2) (at 423.672 121.92 90)
-      (effects (font (size 1.27 1.27)) hide)
-    )
+    (property "Value" "680" (id 1) (at 427.99 123.1899 0)
+      (effects (font (size 1.27 1.27)) (justify left))
+    )
+    (property "Footprint" "Resistor_SMD:R_0603_1608Metric_Pad0.98x0.95mm_HandSolder" (id 2) (at 423.672 121.92 90)
+      (effects (font (size 1.27 1.27)) hide)
+    )

Commit message: Labeled output of U17 (3.5V LDO) 3.5V
Connections:
- net 3.5V: now reaches C58.1, RV2.3, U17.5 (OUT)
Changed lines of the file:
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@@
     (effects (font (size 5 5)) (justify left bottom))
+  )
+  (label "3.5V" (at 468.63 207.01 0)
+    (effects (font (size 1.27 1.27)) (justify left bottom))
   )
   (global_label "LED_Brightness_Control" (shape input) (at 80.01 266.7 0) (fields_autoplaced)

Commit message: Delete unneeded .step (3D-model), .kicad_mod (footprint) and .lib (schematic symbol) files in Project Library folder (AGAIN)
Parts:
- RV1: value 10k_LED_Brightness_Pot -> (none); footprint PTV09A_Pot_Vertical:PTV09 -> (none)
- U18: value NCS333ASQ3T2G -> (none); footprint Package_TO_SOT_SMD:SOT-353_SC-70-5 -> (none)
Changed lines of the file:
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@@
       (effects (font (size 1.27 1.27)) (justify right))
     )
-    (property "Value" "10k_LED_Brightness_Pot" (id 1) (at 355.6 212.0899 0)
+    (property "Value" "" (id 1) (at 355.6 212.0899 0)
       (effects (font (size 1.27 1.27)) (justify right))
     )
-    (property "Footprint" "PTV09A_Pot_Vertical:PTV09" (id 2) (at 358.14 210.82 0)
+    (property "Footprint" "" (id 2) (at 358.14 210.82 0)
       (effects (font (size 1.27 1.27)) hide)
     )
@@
     (in_bom yes) (on_board yes) (fields_autoplaced)
     (property "Reference" "U18" (id 0) (at 533.4 211.201 0))
-    (property "Value" "NCS333ASQ3T2G" (id 1) (at 533.4 213.741 0))
-    (property "Footprint" "Package_TO_SOT_SMD:SOT-353_SC-70-5" (id 2) (at 519.43 215.9 0)
+    (property "Value" "" (id 1) (at 533.4 213.741 0))
+    (property "Footprint" "" (id 2) (at 519.43 215.9 0)
       (effects (font (size 1.27 1.27)) (justify left) hide)
     )

Commit message: Delete unused LED step and fooprint files in the Project library
Parts:
- U10: value LM3915N-1 -> (none); footprint Package_DIP:DIP-18_W7.62mm_Socket -> (none)
Changed lines of the file:
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@@
       (effects (font (size 1.27 1.27)) (justify right))
     )
-    (property "Value" "LM3915N-1" (id 1) (at 118.11 90.1699 90)
+    (property "Value" "" (id 1) (at 118.11 90.1699 90)
       (effects (font (size 1.27 1.27)) (justify right))
     )
-    (property "Footprint" "Package_DIP:DIP-18_W7.62mm_Socket" (id 2) (at 96.52 88.9 0)
+    (property "Footprint" "" (id 2) (at 96.52 88.9 0)
       (effects (font (size 1.27 1.27)) (justify left bottom) hide)
     )

Commit message: Rearraged Power circuitry schematic and made the paper size custom: 180W x 250H
Parts:
- RV1: value (none) -> 10k_LED_Brightness_Pot; footprint (none) -> PTV09A_Pot_Vertical:PTV09
- U10: value (none) -> LM3915N-1; footprint (none) -> Package_DIP:DIP-18_W7.62mm_Socket
- U18: value (none) -> NCS333ASQ3T2G; footprint (none) -> Package_TO_SOT_SMD:SOT-353_SC-70-5
Changed lines of the file:
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@@
       (effects (font (size 1.27 1.27)) (justify right))
     )
-    (property "Value" "" (id 1) (at 355.6 212.0899 0)
-      (effects (font (size 1.27 1.27)) (justify right))
-    )
-    (property "Footprint" "" (id 2) (at 358.14 210.82 0)
+    (property "Value" "10k_LED_Brightness_Pot" (id 1) (at 355.6 212.0899 0)
+      (effects (font (size 1.27 1.27)) (justify right))
+    )
+    (property "Footprint" "PTV09A_Pot_Vertical:PTV09" (id 2) (at 358.14 210.82 0)
       (effects (font (size 1.27 1.27)) hide)
     )
@@
     (in_bom yes) (on_board yes) (fields_autoplaced)
     (property "Reference" "U18" (id 0) (at 533.4 211.201 0))
-    (property "Value" "" (id 1) (at 533.4 213.741 0))
-    (property "Footprint" "" (id 2) (at 519.43 215.9 0)
+    (property "Value" "NCS333ASQ3T2G" (id 1) (at 533.4 213.741 0))
+    (property "Footprint" "Package_TO_SOT_SMD:SOT-353_SC-70-5" (id 2) (at 519.43 215.9 0)
       (effects (font (size 1.27 1.27)) (justify left) hide)
     )
@@
       (effects (font (size 1.27 1.27)) (justify right))
     )
-    (property "Value" "" (id 1) (at 118.11 90.1699 90)
-      (effects (font (size 1.27 1.27)) (justify right))
-    )
-    (property "Footprint" "" (id 2) (at 96.52 88.9 0)
-      (effects (font (size 1.27 1.27)) (justify left bottom) hide)
-    )
+    (property "Value" "LM3915N-1" (id 1) (at 118.11 90.1699 90)
+      (effects (font (size 1.27 1.27)) (justify right))
+    )
+    (property "Footprint" "Package_DIP:DIP-18_W7.62mm_Socket" (id 2) (at 96.52 88.9 0)
+      (effects (font (size 1.27 1.27)) (justify left bottom) hide)
+    )
